Commit message: update nav2_sim : navigation packgae

File: ros2_riscv_car/nav2_sim/src/robot_description/urdf/MicroROS.urdf (robot description, URDF)
Before this commit: robot micro4.0, 9 links, 8 joints
Joints:
- joint yh_Joint: axis 0 -1 0 -> 0 1 0
- joint yq_Joint: axis 0 -1 0 -> 0 1 0
- joint zh_Joint: axis 0 -1 0 -> 0 1 0
- joint zq_Joint: axis 0 -1 0 -> 0 1 0
